File: USB Hub.kicad_sch (KiCad schematic)
At the start: 37 parts, among them J1 Barrel_Jack_MountingPin, J2 UP2-AH-4-TH, J3 USB-A-S-VT, J4 USB-A-S-VT, J5 USB-A-S-VT, J6 10067847-001RLF, U1 USB2514B_Bi, U10 USBLC6-2SC6, U11 USBLC6-2SC6, U12 D1213A-04V-7, U13 D1213A-04V-7, U2 MIC5504-3.3YM5, U3 MIC2095-2YMT-TR, U4 MIC2095-2YMT-TR, U5 MIC2095-2YMT-TR, U6 MIC2095-2YMT-TR, U7 GL823K-HCY04, U8 USBLC6-2SC6, U9 USBLC6-2SC6, Y1 25MHz

Commit message: First revision of schematic
Parts:
- removed C4, C5, C6: C_Polarized_Small_US, symbol Device:C_Polarized_Small_US
- removed D3: LED, symbol Device:LED
- removed J2: UP2-AH-4-TH, UP2-AH-4-TH:CUI_UP2-AH-4-TH, symbol Custom Symbols:UP2-AH-4-TH
- removed J3, J4, J5: USB-A-S-VT, Custom Footprints:CONN_USB-A-S-VT_ADM, symbol Custom Symbols:USB-A-S-VT
- removed U3, U4, U5, U6: MIC2095-2YMT-TR, TMLF-6_MT_MCH, symbol Custom Symbols:MIC2095-2YMT-TR
- added C1, C12, C2: 2u2, Capacitor_SMD:C_0805_2012Metric_Pad1.18x1.45mm_HandSolder, symbol Device:C_Small
- added C10, C13, C14, C15, C16, C17, C18, C19, C20, C21, C23, C7, C8: 100n, Capacitor_SMD:C_0805_2012Metric_Pad1.18x1.45mm_HandSolder, symbol Device:C_Small
- added C11, C22, C24, C25, C26, C9: 1uF, Capacitor_SMD:C_0805_2012Metric_Pad1.18x1.45mm_HandSolder, symbol Device:C_Small
- added C28, C29: 100u, Capacitor_THT:CP_Radial_D5.0mm_P2.00mm, symbol Device:C_Polarized_Small_US
- added C30: 4u7, Capacitor_SMD:C_0805_2012Metric_Pad1.18x1.45mm_HandSolder, symbol Device:C_Small
- added D1, D5: LED, LED_SMD:LED_0603_1608Metric_Pad1.05x0.95mm_HandSolder, symbol Device:LED
- added FB1: 120R, Inductor_SMD:L_0805_2012Metric_Pad1.05x1.20mm_HandSolder, symbol Device:FerriteBead_Small
- added J2: 10118193-0001LF, Custom Footprints:AMPHENOL_10118193-0001LF, symbol Custom Symbols:10118193-0001LF
- added J4, J5, J6: UE27AC5410H, Custom Footprints:AMPHENOL_UE27AC5410H, symbol Custom Symbols:UE27AC5410H
- added JP1: ~, Jumper:SolderJumper-2_P1.3mm_Open_Pad1.0x1.5mm, symbol Jumper:SolderJumper_2_Open
- added R1, R10, R2, R4, R5, R6, R7, R8: 100k, Resistor_SMD:R_0805_2012Metric_Pad1.20x1.40mm_HandSolder, symbol Device:R_Small_US
- added R11: 12k, Resistor_SMD:R_0805_2012Metric_Pad1.20x1.40mm_HandSolder, symbol Device:R_Small_US
- added R12, R13, R14, R16, R9: 10k, Resistor_SMD:R_0805_2012Metric_Pad1.20x1.40mm_HandSolder, symbol Device:R_Small_US
- added R15, R18, R19, R20, R21: 330R, Resistor_SMD:R_0805_2012Metric_Pad1.20x1.40mm_HandSolder, symbol Device:R_Small_US
- added R17: 15k, Resistor_SMD:R_0805_2012Metric_Pad1.20x1.40mm_HandSolder, symbol Device:R_Small_US
- added R3: 1M, Resistor_SMD:R_0805_2012Metric, symbol Device:R_Small_US
- added U1: TPS2116DRLR, Custom Footprints:SOTFL50P160X60-8N, symbol Custom Symbols:TPS2116DRLR
- added U10, U11, U12, U8: MIC2005A-1YM5-TR, Package_TO_SOT_SMD:SOT-23-5_HandSoldering, symbol Custom Symbols:MIC2005A-1YM5-TR
- added U3: M24C02-WMN, Package_SO:SOIC-8_3.9x4.9mm_P1.27mm, symbol Memory_EEPROM:M24C02-WMN
- added U5: 74LVC1G86, Package_TO_SOT_SMD:SOT-353_SC-70-5_Handsoldering, symbol 74xGxx:74LVC1G86
- added U6: 74LVC1G04, Package_TO_SOT_SMD:SOT-23-5_HandSoldering, symbol 74xGxx:74LVC1G04
- C27: renamed from C3; value C_Polarized_Small_US -> 100u; footprint (none) -> Capacitor_THT:CP_Radial_D5.0mm_P2.00mm
- C3: renamed from C1; value C_Small -> 2u2; footprint Capacitor_SMD:C_0805_2012Metric -> Capacitor_SMD:C_0805_2012Metric_Pad1.18x1.45mm_HandSolder
- C4: renamed from C7; footprint Capacitor_SMD:C_0603_1608Metric -> Capacitor_SMD:C_0603_1608Metric_Pad1.08x0.95mm_HandSolder
- C5: renamed from C2; value C_Small -> 2u2; footprint (none) -> Capacitor_SMD:C_0805_2012Metric_Pad1.18x1.45mm_HandSolder
- C6: renamed from C8; footprint Capacitor_SMD:C_0603_1608Metric -> Capacitor_SMD:C_0603_1608Metric_Pad1.08x0.95mm_HandSolder
- D2, D4: footprint (none) -> LED_SMD:LED_0603_1608Metric_Pad1.05x0.95mm_HandSolder
- D3: renamed from D1; footprint LED_SMD:LED_0603_1608Metric -> LED_SMD:LED_0603_1608Metric_Pad1.05x0.95mm_HandSolder
- FB2: renamed from FB1; value FerriteBead_Small -> 120R; footprint Inductor_SMD:L_0805_2012Metric -> Inductor_SMD:L_0805_2012Metric_Pad1.05x1.20mm_HandSolder
- U15: renamed from U8; footprint Package_TO_SOT_SMD:SOT-23-6_Handsoldering -> Package_TO_SOT_SMD:SOT-23-6
- U16: renamed from U9; footprint Package_TO_SOT_SMD:SOT-23-6_Handsoldering -> Package_TO_SOT_SMD:SOT-23-6
- U17: renamed from U10; footprint Package_TO_SOT_SMD:SOT-23-6_Handsoldering -> Package_TO_SOT_SMD:SOT-23-6
- U2: renamed from U11; footprint Package_TO_SOT_SMD:SOT-23-6_Handsoldering -> Package_TO_SOT_SMD:SOT-23-6
- renumbered J6 to J3, U12 to U13, U13 to U14, U2 to U4, U1 to U7, U7 to U9
Connections:
- net GND: now also C27.2, C3.2, C4.2, C5.2, C6.2, J1.2, J1.MP (MountPin), J3.10 (CD), J3.11 (WP), J3.12 (GND), J3.13 (GND), J3.3 (VSS), J3.6 (VSS), U13.2 (GND), U14.2 (GND), U15.2 (GND), U16.2 (GND), U17.2 (GND), U2.2 (GND), U4.2 (GND), U9.1 (VSS), U9.11 (GPIO), U9.14 (VSS), C1.2, C10.2, C11.2, C12.2, C13.2, C14.2, C15.2, C16.2, C17.2, C18.2, C19.2, C2.2, C20.2, C21.2, C22.2, C23.2, C24.2, C25.2, C26.2, C28.2, C29.2, C30.2, C7.2, C8.2, C9.2, J2.5 (GND), J2.S1 (SHIELD), J2.S2 (SHIELD__1), J2.S3 (SHIELD__2), J2.S4 (SHIELD__3), J2.S5 (SHIELD__4), J2.S6 (SHIELD__5), J4.4 (GND), J4.SH1 (SHIELD), J4.SH2 (SHIELD__1), J5.4 (GND), J5.SH1 (SHIELD), J5.SH2 (SHIELD__1), J6.4 (GND), J6.SH1 (SHIELD), J6.SH2 (SHIELD__1), R1.1, R10.2, R11.1, R15.1, R17.2, R18.1, R19.1, R20.1, R21.1, R6.2, R7.2, R8.2, U1.1 (GND), U10.2 (GND), U11.2 (GND), U12.2 (GND), U3.1 (E0), U3.2 (E1), U3.3 (E2), U3.4 (VSS), U5.3 (GND), U6.3 (GND), U8.2 (GND)
- net at C27.1: now also D3.2 (A), U15.5 (VBUS), J4.1 (VCC), U10.5 (VOUT)
- net 5V_HOST_FILTER: now reaches C5.1
- net 5V_HOST_FILTER: now also FB2.2, R5.2, U1.6 (VIN2)
- net at U2.1 (I/O1): now also J2.2 (D-)
- net at U2.3 (I/O2): now also J2.3 (D+)
- net USB_UP_D+: now reaches U2.4 (I/O2)
- net USB_UP_D+: now also U7.31 (USBDP_UP)
- net 5V_HOST: now reaches U2.5 (VBUS)
- net 5V_HOST: now also C3.1, FB2.1, J2.1 (VUSB)
- net USB_UP_D-: now reaches U2.6 (I/O1)
- net USB_UP_D-: now also U7.30 (USBDM_UP)
- net 5V: now reaches U4.1 (VIN)
- net 5V: now also C20.1, C21.1, C22.1, C24.1, C25.1, C26.1, C9.1, U1.2 (VOUT), U1.7 (VOUT), U10.1 (VIN), U11.1 (VIN), U12.1 (VIN), U5.5 (VCC), U6.5 (VCC), U8.1 (VIN)
- net VBUS_DET: now reaches U4.3 (EN)
- net VBUS_DET: now also U7.27 (VBUS_DET), R5.1, R6.1
- net 3V3: now reaches U4.5 (VOUT)
- net 3V3: now also U7.10 (VDDA33), U7.15 (VDD33), U7.23 (VDD33), U7.29 (VDDA33), U7.36 (VDDA33), U7.5 (VDDA33), C11.1, C12.1, C13.1, C14.1, C15.1, C16.1, C17.1, C18.1, C19.1, D1.2 (A), JP1.1 (A), R12.1, R13.1, R14.2, U3.7 (~{WC}), U3.8 (VCC)
- net at D2.1 (K): now also R18.2
- net at D2.2 (A): now also U9.12 (LED)
- net at J3.1 (CD/DAT3): now also U9.6 (D3)
- net at J3.2 (CMD): now also U13.1 (CH1), U9.5 (CMD)
- net 3V3_SD: now reaches J3.4 (VDD)
- net 3V3_SD: now also U13.5 (VPP), U14.4 (CH3), U14.5 (VPP), U9.8 (PMOS), C30.1
- net at J3.5 (CLK): now also U13.3 (CH2), U9.4 (CLK)
- net at J3.7 (DAT0): now also U14.1 (CH1), U9.3 (D0)
- net at J3.8 (DAT1): now also U13.6 (CH4), U9.2 (D1)
- net at J3.9 (DAT2): now also U13.4 (CH3), U9.7 (D2)
- net at Y1.1: now also C4.1, U7.33 (XTALIN/CLKIN), R3.1
- net at Y1.2: now also C6.1, U7.32 (XTALOUT), R3.2
- net USB1_D-: now reaches U7.1 (USBDM_DN1/PRT_DIS_M1)
- net USB1_D-: now also U15.1 (I/O1)
- net USB1_EN: now reaches U7.12 (PRTPWR1/BC_EN1)
- net USB1_EN: now also U10.3 (EN)
- net USB1_OC: now reaches U7.13 (OCS_N1)
- net USB1_OC: now also U10.4 (nFAULT)
- net at U7.14 (CRFILT): now also C8.1
- net USB2_EN: now reaches U7.16 (PRTPWR2/BC_EN2)
- net USB2_EN: now also U11.3 (EN)
- net USB2_OC: now reaches U7.17 (OCS_N2)
- net USB2_OC: now also U11.4 (nFAULT)
- net USB3_EN: now reaches U7.18 (PRTPWR3/BC_EN3)
- net USB3_EN: now also U12.3 (EN)
- net USB3_OC: now reaches U7.19 (OCS_N3)
- net USB3_OC: now also U12.4 (nFAULT)
- net USB1_D+: now reaches U7.2 (USBDP_DN1/PRT_DIS_P1)
- net USB1_D+: now also U15.3 (I/O2)
- net USB4_EN: now reaches U7.20 (PRTPWR4/BC_EN4)
- net USB4_EN: now also U8.3 (EN)
- net USB4_OC: now reaches U7.21 (OCS_N4)
- net USB4_OC: now also U8.4 (nFAULT)
- net EEPROM_SDA: now reaches U7.22 (SDA/SMBDATA/NON_REM1)
- net EEPROM_SDA: now also R13.2, R8.1, U3.6 (SCL)
- net EEPROM_SCL: now reaches U7.24 (SCL/SMBCLK/CFG_SEL0)
- net EEPROM_SCL: now also R12.2, R7.1, U3.5 (SDA)
- net at U7.25 (HS_IND/CFG_SEL1): now also R14.1
- net RESET: now reaches U7.26 (RESET_N)
- net RESET: now also JP1.2 (B), R16.2, R17.1
- net LOCAL_PWR: now reaches U7.28 (SUSP_IND/LOCAL_PWR/NON_REM0)
- net LOCAL_PWR: now also R10.1, R4.1, R9.2, U1.8 (ST), U5.1
- net USB2_D-: now reaches U7.3 (USBDM_DN2/PRT_DIS_M2)
- net USB2_D-: now also U16.1 (I/O1)
- net at U7.34 (PLLFILT): now also C7.1
- net at U7.35 (RBIAS): now also R11.2
- net USB2_D+: now reaches U7.4 (USBDP_DN2/PRT_DIS_P2)
- net USB2_D+: now also U16.3 (I/O2)
- net USB3_D-: now reaches U7.6 (USBDM_DN3/PRT_DIS_M3)
- net USB3_D-: now also U17.1 (I/O1)
- net USB3_D+: now reaches U7.7 (USBDP_DN3/PRT_DIS_P3)
- net USB3_D+: now also U17.3 (I/O2)
- net USB4_D-: now reaches U7.8 (USBDM_DN4/PRT_DIS_M4)
- net USB4_D-: now also U9.16 (D-)
- net USB4_D+: now reaches U7.9 (USBDP_DN4/PRT_DIS_P4)
- net USB4_D+: now also U9.15 (D+)
- net at D3.1 (K): now also R19.2
- net at D4.1 (K): now also R20.2
- net at D4.2 (A): now also U16.5 (VBUS), C28.1, J5.1 (VCC), U11.5 (VOUT)
- net at U16.4 (I/O2): now also J5.3 (D+)
- net at U16.6 (I/O1): now also J5.2 (D-)
- net at U15.4 (I/O2): now also J4.3 (D+)
- net at U15.6 (I/O1): now also J4.2 (D-)
- net at U9.10 (5V): now also C23.1, U8.5 (VOUT)
- net at U17.4 (I/O2): now also J6.3 (D+)
- net at U17.5 (VBUS): now also C29.1, D5.2 (A), J6.1 (VCC), U12.5 (VOUT)
- net at U17.6 (I/O1): now also J6.2 (D-)
- net 5V_IN: now reaches J1.1
- net 5V_IN: now also C1.1, FB1.1
- new net: R1.2, R2.1, U1.4 (PR1)
- new net: C10.1, R9.1, U5.2
- new net: U5.4, U6.2
- new net: R16.1, U6.4
- new net: D5.1 (K), R21.2
- new net: D1.1 (K), R15.2
- new net 5V_FILTER: C2.1, FB1.2, R2.2, R4.2, U1.3 (VIN1), U1.5 (MODE)
- no-connect marks 0 -> 6
Other:
- moved on the sheet: C27, C3, C4, C5, C6, D3, FB2, H1, H2, H3, H4, J1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

Commit message: first layout revision + some schematic rearrangements
Parts:
- removed Y1: 25MHz, Crystal:Crystal_HC49-4H_Vertical, symbol Device:Crystal
- added C10: 100n, Capacitor_SMD:C_0805_2012Metric_Pad1.18x1.45mm_HandSolder, symbol Device:C_Small
- added C12: 10n, Capacitor_SMD:C_0805_2012Metric_Pad1.18x1.45mm_HandSolder, symbol Device:C_Small
- added JP2, JP3, JP4: ~, Jumper:SolderJumper-2_P1.3mm_Open_Pad1.0x1.5mm, symbol Jumper:SolderJumper_2_Open
- added Y1: ECS-240, Custom Footprints:XTAL_ECS-240-12-37B-CKY-TR, symbol Custom Symbols:ECS-240-12-37B-CKY-TR
- C4, C6: value 8pF -> 16p
- C8: value 100n -> 10n
- H1, H2, H3, H4: footprint (none) -> MountingHole:MountingHole_3.2mm_M3_DIN965_Pad
- J1: footprint Connector_BarrelJack:BarrelJack_GCT_DCJ200-10-A_Horizontal -> Custom Footprints:BarrelJack_GCT_DCJ200-10-A_Horizontal
- renumbered C10 to C11, C11 to C13, C12 to C14, C13 to C15, C14 to C16, C15 to C17, C16 to C18, C17 to C19, C18 to C20, C19 to C21, C20 to C22, C21 to C23, C22 to C24, C23 to C25, C24 to C26, C25 to C27, C26 to C28, C27 to C29, C28 to C30, C29 to C31, C30 to C32, R12 to R10, R8 to R11, R13 to R12, R10 to R13, R9 to R7, R7 to R8, R11 to R9
Connections:
- net 3V3_SD: now also U13.1 (CH1), JP3.1 (A); no longer U14.4 (CH3)
- net GND: now also J1.3 (MountPin), U7.11 (TEST), C10.2, C12.2, JP4.1 (A), Y1.2 (GND), Y1.4 (GND); no longer J1.MP (MountPin), R18.1
- net LOCAL_PWR: now also JP2.1 (A); no longer R13.1, U7.28 (SUSP_IND/LOCAL_PWR/NON_REM0)
- net USB1_D+: now also U9.15 (D+); no longer U15.3 (I/O2)
- net USB1_D-: now also U9.16 (D-); no longer U15.1 (I/O1)
- net USB1_EN: now also U8.3 (EN); no longer U10.3 (EN)
- net USB1_OC: now also U8.4 (nFAULT); no longer U10.4 (nFAULT)
- net USB2_D+: now also U17.3 (I/O2); no longer U16.3 (I/O2)
- net USB2_D-: now also U17.1 (I/O1); no longer U16.1 (I/O1)
- net USB2_EN: now also U12.3 (EN); no longer U11.3 (EN)
- net USB2_OC: now also U12.4 (nFAULT); no longer U11.4 (nFAULT)
- net USB3_D+: now also U16.3 (I/O2); no longer U17.3 (I/O2)
- net USB3_D-: now also U16.1 (I/O1); no longer U17.1 (I/O1)
- net USB3_EN: now also U11.3 (EN); no longer U12.3 (EN)
- net USB3_OC: now also U11.4 (nFAULT); no longer U12.4 (nFAULT)
- net USB4_D+: now also U15.3 (I/O2); no longer U9.15 (D+)
- net USB4_D-: now also U15.1 (I/O1); no longer U9.16 (D-)
- net USB4_EN: now also U10.3 (EN); no longer U8.3 (EN)
- net USB4_OC: now also U10.4 (nFAULT); no longer U8.4 (nFAULT)
- net at J3.1 (CD/DAT3), U9.6 (D3): now also U13.6 (CH4)
- net at J3.2 (CMD), U9.5 (CMD): no longer U13.1 (CH1)
- net at J3.5 (CLK), U9.4 (CLK): now also U14.6 (CH4); no longer U13.3 (CH2)
- net at J3.7 (DAT0), U9.3 (D0): now also U14.3 (CH2); no longer U14.1 (CH1)
- net at J3.8 (DAT1), U9.2 (D1): now also U14.1 (CH1); no longer U13.6 (CH4)
- net at C4.1, R3.1, U7.33 (XTALIN/CLKIN): now also Y1.1 (IN/OUT)
- net at C6.1, R3.2, U7.32 (XTALOUT): now also Y1.3 (OUT/IN)
- net at U7.14 (CRFILT): now also C10.1, C12.1; no longer C8.1
- net at C7.1, U7.34 (PLLFILT): now also C8.1
- new net: JP2.2 (B), R13.1, U7.28 (SUSP_IND/LOCAL_PWR/NON_REM0)
- new net: JP3.2 (B), JP4.2 (B), R18.1
- no-connect marks 6 -> 5
Other:
- moved on the sheet: C4, C6, C7, R11, R13, R14, R3, R8, U7

Commit message: Fixed reference designator silkscreen and add copper pours to power section
Parts:
- removed Y1: ECS-240, Custom Footprints:XTAL_ECS-240-12-37B-CKY-TR, symbol Custom Symbols:ECS-240-12-37B-CKY-TR
- added Y1: Crystal, Custom Footprints:XTAL_HC49P488W43L1150T466H350, symbol Device:Crystal
- C4, C6: value 16p -> 8p
Connections:
- net at C6.1, R3.2, U7.32 (XTALOUT): now also Y1.2
- net at C4.1, R3.1, U7.33 (XTALIN/CLKIN): now also Y1.1
Changed lines of the file:
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@@
 	)
 	(junction
-		(at 110.49 299.72)
-		(diameter 0)
-		(color 0 0 0 0)
-	)
-	(junction
 		(at 97.79 283.21)
 		(diameter 0)
@@
 	(wire
 		(pts
-			(xy 107.95 295.91) (xy 107.95 299.72)
-		)
-		(stroke
-			(width 0)
-			(type default)
-		)
-	)
-	(wire
-		(pts
 			(xy 138.43 87.63) (xy 151.13 87.63)
 		)
@@
 	(wire
 		(pts
-			(xy 110.49 295.91) (xy 110.49 299.72)
-		)
-		(stroke
-			(width 0)
-			(type default)
-		)
-	)
-	(wire
-		(pts
 			(xy 179.07 74.93) (xy 179.07 78.74)
 		)
@@
 	(wire
 		(pts
-			(xy 107.95 299.72) (xy 110.49 299.72)
-		)
-		(stroke
-			(width 0)
-			(type default)
-		)
-	)
-	(wire
-		(pts
 			(xy 228.6 214.63) (xy 226.06 214.63)
 		)
@@
 	(wire
 		(pts
-			(xy 97.79 283.21) (xy 99.06 283.21)
+			(xy 97.79 283.21) (xy 105.41 283.21)
 		)
 		(stroke
@@
 	(wire
 		(pts
-			(xy 110.49 299.72) (xy 120.65 299.72)
+			(xy 107.95 299.72) (xy 120.65 299.72)
 		)
 		(stroke
@@
 	(wire
 		(pts
+			(xy 113.03 283.21) (xy 120.65 283.21)
+		)
+		(stroke
+			(width 0)
+			(type default)
+		)
+	)
+	(wire
+		(pts
 			(xy 454.66 209.55) (xy 466.09 209.55)
 		)
@@
 	(wire
 		(pts
-			(xy 119.38 283.21) (xy 120.65 283.21)
-		)
-		(stroke
-			(width 0)
-			(type default)
-		)
-	)
-	(wire
-		(pts
 			(xy 508 256.54) (xy 495.3 256.54)
 		)
@@
 	)
 	(symbol
-		(lib_id "Custom Symbols:ECS-240-12-37B-CKY-TR")
-		(at 114.3 285.75 0)
-		(unit 1)
-		(exclude_from_sim no)
-		(in_bom yes)
-		(on_board yes)
-		(dnp no)
-		(fields_autoplaced yes)
-		(property "Reference" "Y1"
-			(at 109.22 275.59 0)
-			(effects
-				(font
-					(size 1.27 1.27)
-				)
-			)
-		)
-		(property "Value" "ECS-240"
-			(at 109.22 278.13 0)
-			(effects
-				(font
-					(size 1.27 1.27)
-				)
-			)
-		)
-		(property "Footprint" "Custom Footprints:XTAL_ECS-240-12-37B-CKY-TR"
-			(at 152.4 294.386 0)
-			(effects
-				(font
-					(size 1.27 1.27)
-				)
-				(justify bottom)
-				(hide yes)
-			)
-		)
-		(property "Datasheet" ""
-			(at 114.3 285.75 0)
-			(effects
-				(font
-					(size 1.27 1.27)
-				)
-				(hide yes)
-			)
-		)
-		(property "Description" ""
-			(at 114.3 285.75 0)
-			(effects
-				(font
-					(size 1.27 1.27)
-				)
-				(hide yes)
-			)
-		)
-		(pin "3"
-		)
-		(pin "2"
-		)
-		(pin "1"
-		)
-		(pin "4"
-		)
-		(instances
-			(project ""
-				(path "/c61904c1-a3bf-47f0-94e4-e1e35430634d"
-					(reference "Y1")
-					(unit 1)
-				)
-			)
-		)
-	)
-	(symbol
 		(lib_id "Device:C_Polarized_Small_US")
 		(at 454.66 247.65 0)
@@
 			)
 		)
-		(property "Value" "16p"
+		(property "Value" "8p"
 			(at 95.25 293.3762 0)
 			(effects
@@
 			)
 		)
-		(property "Value" "16p"
+		(property "Value" "8p"
 			(at 123.19 293.3762 0)
 			(effects
@@
 					(unit 1)
 				)
+			)
+		)
+	)
+	(symbol
+		(lib_id "Device:Crystal")
+		(at 109.22 283.21 0)
+		(unit 1)
+		(exclude_from_sim no)
+		(in_bom yes)
+		(on_board yes)
+		(dnp no)
+		(fields_autoplaced yes)
+		(property "Reference" "Y1"
+			(at 109.22 275.59 0)
+			(effects
+				(font
+					(size 1.27 1.27)
+				)
+			)
+		)
+		(property "Value" "Crystal"
+			(at 109.22 278.13 0)
+			(effects
+				(font
+					(size 1.27 1.27)
+				)
+			)
+		)
+		(property "Footprint" "Custom Footprints:XTAL_HC49P488W43L1150T466H350"
+			(at 109.22 283.21 0)
+			(effects
+				(font
+					(size 1.27 1.27)
+				)
+				(hide yes)
+			)
+		)
+		(property "Datasheet" "~"
+			(at 109.22 283.21 0)
+			(effects
+				(font
+					(size 1.27 1.27)
+				)
+				(hide yes)
+			)
+		)
+		(property "Description" "Two pin crystal"
+			(at 109.22 283.21 0)
+			(effects
+				(font
+					(size 1.27 1.27)
+				)
+				(hide yes)
+			)
+		)
+		(pin "2"
+		)
+		(pin "1"
+		)
+		(instances
+			(project ""
+				(path "/c61904c1-a3bf-47f0-94e4-e1e35430634d"
+					(reference "Y1")
+					(unit 1)
+				)

Commit message: v2 of USB Hub
Parts:
- removed C11, C22: 100n, Capacitor_SMD:C_0805_2012Metric_Pad1.18x1.45mm_HandSolder, symbol Device:C_Small
- removed JP1, JP3, JP4: ~, Jumper:SolderJumper-2_P1.3mm_Open_Pad1.0x1.5mm, symbol Jumper:SolderJumper_2_Open
- removed R16, R7: 10k, Resistor_SMD:R_0805_2012Metric_Pad1.20x1.40mm_HandSolder, symbol Device:R_Small_US
- removed R17: 15k, Resistor_SMD:R_0805_2012Metric_Pad1.20x1.40mm_HandSolder, symbol Device:R_Small_US
- removed U5: 74LVC1G86, Package_TO_SOT_SMD:SOT-353_SC-70-5_Handsoldering, symbol 74xGxx:74LVC1G86
- removed U6: 74LVC1G04, Package_TO_SOT_SMD:SOT-23-5_HandSoldering, symbol 74xGxx:74LVC1G04
- added C24: 2u2, Capacitor_SMD:C_0805_2012Metric_Pad1.18x1.45mm_HandSolder, symbol Device:C_Small
- added C28: 100n, Capacitor_SMD:C_0805_2012Metric_Pad1.18x1.45mm_HandSolder, symbol Device:C_Small
- added JP2: SolderJumper_3_Open, Jumper:SolderJumper-3_P2.0mm_Open_TrianglePad1.0x1.5mm_NumberLabels, symbol Jumper:SolderJumper_3_Open
- added R15: 10k, Resistor_SMD:R_0805_2012Metric_Pad1.20x1.40mm_HandSolder, symbol Device:R_Small_US
- added R5: 100k, Resistor_SMD:R_0805_2012Metric_Pad1.20x1.40mm_HandSolder, symbol Device:R_Small_US
- added SW1: 1825910-6, Library:SW4_1825910-B_TEC, symbol Custom Symbols1:1825910-6
- added TP1: GND, TestPoint:TestPoint_THTPad_D4.0mm_Drill2.0mm, symbol Connector:TestPoint
- added TP2: SDA, TestPoint:TestPoint_THTPad_2.0x2.0mm_Drill1.0mm, symbol Connector:TestPoint
- added TP3: SCL, TestPoint:TestPoint_THTPad_2.0x2.0mm_Drill1.0mm, symbol Connector:TestPoint
- added TP4: 3V3_SD, TestPoint:TestPoint_THTPad_2.0x2.0mm_Drill1.0mm, symbol Connector:TestPoint
- C23: value 100n -> 4u7
- C29, C30, C31: value 100u -> 120uF
- U5: renamed from U7; footprint Package_DFN_QFN:QFN-36-1EP_6x6mm_P0.5mm_EP3.7x3.7mm -> Library:QFN-36-1EP_6x6mm_P0.5mm_EP3.7x3.7mm_ThermalVias
- renumbered C9 to C10, C10 to C11, C16 to C15, C17 to C16, C18 to C17, C19 to C18, C20 to C19, C21 to C20, C24 to C21, C25 to C22, C26 to C25, C27 to C26, C28 to C27, C15 to C5, C5 to C6, C6 to C7, C7 to C8, C8 to C9, J4 to J3, J5 to J4, J6 to J5, J3 to J6, JP2 to JP1, R15 to R16, R18 to R17, R19 to R18, R20 to R19, R21 to R20, R5 to R6, R6 to R7, U12 to U10, U13 to U11, U14 to U12, U15 to U13, U16 to U14, U17 to U15, U8 to U6, U9 to U7, U10 to U8, U11 to U9
Connections:
- net 3V3: now also JP2.3 (B), R15.1
- net 3V3_SD: now also R17.1, U7.13 (VDDA), U7.9 (VDD), C24.1, C28.1, TP4.1; no longer C32.1, J6.4 (VDD), U11.1 (CH1), U11.5 (VPP), U12.5 (VPP), U7.8 (PMOS)
- net 5V: no longer C23.1
- net EEPROM_SCL: now also R12.2, U3.6 (SCL), TP3.1; no longer R10.2, U3.5 (SDA)
- net EEPROM_SDA: now also R10.2, U3.5 (SDA), TP2.1; no longer R12.2, U3.6 (SCL)
- net GND: now also C24.2, C28.2, SW1.1, SW1.2, TP1.1; no longer J6.10 (CD)
- net LOCAL_PWR: now also R5.2; no longer U1.8 (ST)
- net RESET: now also R15.2, SW1.3, SW1.4
- net at D2.1 (K): now also U7.12 (LED); no longer R17.2
- net at D2.2 (A): now also R17.2; no longer U7.12 (LED)
- net at C22.1, U6.5 (VOUT), U7.10 (5V): now also C23.1
- new net: R5.1, U1.8 (ST)
- new net: JP2.1 (A), U7.8 (PMOS)
- new net 3V3_PMOS: C32.1, J6.4 (VDD), JP2.2 (C), U11.1 (CH1), U11.5 (VPP), U12.5 (VPP)
- no-connect marks 5 -> 4
Other:
- moved on the sheet: C21, C22, C32, C4, C5, C7, D2, J6, R17, R3, R4, U11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
